File: HBroBil.kicad_sch (KiCad schematic)
At the start: 14 parts, among them J1 Conn_01x07_Male, J2 Conn_02x04_Odd_Even

Commit message: Comparator component
Parts:
- removed ComperatorSocket1: Conn_02x04_Counter_Clockwise, Connector_PinSocket_1.27mm:PinSocket_2x04_P1.27mm_Vertical, symbol Connector_Generic:Conn_02x04_Counter_Clockwise
- added IC1: MCP6542-I_P, DIP781W56P254L950H533Q8N, symbol MCP6542-I_P:MCP6542-I_P
Connections:
- net 5V: now also IC1.8 (VDD)
- net at NPN2.1 (G), PNP2.1 (G): now also IC1.7 (OUTB)
- net at Auto/Man1.2, NPN1.1 (G), PNP1.1 (G): now also IC1.6 (VINB-)
- net at R1.2, R2.1: now also IC1.5 (VINB+)

Commit message: Finito
Parts:
- removed J2: Conn_02x04_Odd_Even, symbol Connector_Generic:Conn_02x04_Odd_Even
- added FlybackNPN1, FlybackNPN2, FlybackPNP1, FlybackPNP2: R_Small_US, Resistor_THT:R_Axial_DIN0204_L3.6mm_D1.6mm_P5.08mm_Horizontal, symbol Device:R_Small_US
- added InvertedLamp1, Lamp1: Lamp, Resistor_THT:R_Axial_DIN0204_L3.6mm_D1.6mm_P5.08mm_Horizontal, symbol Device:Lamp
- added R3, R4: R, Resistor_THT:R_Axial_DIN0204_L3.6mm_D1.6mm_P5.08mm_Horizontal, symbol Device:R
- renumbered ManuelHastighed1 to PotentioMTR1
Connections:
- net 6V: now also FlybackPNP1.1, FlybackPNP2.1
- net MTR +: now also FlybackNPN1.2, FlybackPNP1.2
- net MTR -: now also FlybackNPN2.2, FlybackPNP2.2
- net at NPN2.1 (G), PNP2.1 (G): now also InvertedLamp1.1 (-); no longer IC1.7 (OUTB)
- net at NPN1.3 (S), NPN2.3 (S), NPN3.2 (D): now also FlybackNPN1.1, FlybackNPN2.1
- net at NPN1.1 (G), PNP1.1 (G): now also Lamp1.1 (-); no longer Auto/Man1.2, IC1.6 (VINB-)
- new net: IC1.7 (OUTB), R4.1
- new net: InvertedLamp1.2 (+), R4.2
- new net: Auto/Man1.2, IC1.6 (VINB-), R3.1
- new net: Lamp1.2 (+), R3.2

Commit message: fixs
Connections:
- net GND is gone; now on net GNDREF: R2.2
- net GNDREF: now also PotentioMTR1.3
Changed lines of the file:
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@@
     (pin "3")
+  )
+  (symbol (lib_id "power:GNDREF") (at 102.87 82.55 0) (unit 1)
+    (in_bom yes) (on_board yes) (fields_autoplaced)
+    (property "Reference" "#PWR0105" (id 0) (at 102.87 88.9 0)
+      (effects (font (size 1.27 1.27)) hide)
+    )
+    (property "Value" "GNDREF" (id 1) (at 102.87 87.63 0))
+    (property "Footprint" "" (id 2) (at 102.87 82.55 0)
+      (effects (font (size 1.27 1.27)) hide)
+    )
+    (property "Datasheet" "" (id 3) (at 102.87 82.55 0)
+      (effects (font (size 1.27 1.27)) hide)
+    )
+    (pin "1")
   )
   (symbol (lib_id "Device:R_Small_US") (at 104.14 142.24 90) (unit 1)
@@
     (pin "2")
   )
+  (symbol (lib_id "power:GNDREF") (at 106.68 142.24 90) (unit 1)
+    (in_bom yes) (on_board yes) (fields_autoplaced)
+    (property "Reference" "#PWR0104" (id 0) (at 113.03 142.24 0)
+      (effects (font (size 1.27 1.27)) hide)
+    )
+    (property "Value" "GNDREF" (id 1) (at 110.49 142.2399 90)
+      (effects (font (size 1.27 1.27)) (justify right))
+    )
+    (property "Footprint" "" (id 2) (at 106.68 142.24 0)
+      (effects (font (size 1.27 1.27)) hide)
+    )
+    (property "Datasheet" "" (id 3) (at 106.68 142.24 0)
+      (effects (font (size 1.27 1.27)) hide)
+    )
+    (pin "1")
+  )
   (symbol (lib_id "100SP1T1B4M2QE:100SP1T1B4M2QE") (at 110.49 96.52 180) (unit 1)
     (in_bom yes) (on_board yes) (fields_autoplaced)
@@
     (pin "2")
     (pin "3")
-  )
-  (symbol (lib_id "power:GND") (at 106.68 142.24 90) (unit 1)
-    (in_bom yes) (on_board yes) (fields_autoplaced)
-    (property "Reference" "#PWR0105" (id 0) (at 113.03 142.24 0)
-      (effects (font (size 1.27 1.27)) hide)
-    )
-    (property "Value" "GND" (id 1) (at 111.76 142.24 0))
-    (property "Footprint" "" (id 2) (at 106.68 142.24 0)
-      (effects (font (size 1.27 1.27)) hide)
-    )
-    (property "Datasheet" "" (id 3) (at 106.68 142.24 0)
-      (effects (font (size 1.27 1.27)) hide)
-    )
-    (pin "1")
   )
   (symbol (lib_id "Device:Lamp") (at 124.46 114.3 90) (unit 1)
@@
       (reference "#PWR0103") (unit 1) (value "GNDREF") (footprint "")
     )
-    (path "/a02be8e7-7b00-456f-a319-a1a12d419540"
-      (reference "#PWR0105") (unit 1) (value "GND") (footprint "")
+    (path "/9d159183-986f-42b2-9b59-de7d216f55de"
+      (reference "#PWR0104") (unit 1) (value "GNDREF") (footprint "")
+    )
+    (path "/2fa0d964-252a-4916-986a-fc99c14c8137"
+      (reference "#PWR0105") (unit 1) (value "GNDREF") (footprint "")
     )
     (path "/f4ec7ea6-8beb-43cb-a9fc-1096ac2d6bfa"

Commit message: lAST FIXES
Parts:
- FlybackNPN1, FlybackNPN2, FlybackPNP1, FlybackPNP2, R1, R2, R3, R4: footprint Resistor_THT:R_Axial_DIN0204_L3.6mm_D1.6mm_P5.08mm_Horizontal -> Resistor_THT:R_Axial_DIN0204_L3.6mm_D1.6mm_P7.62mm_Horizontal
- InvertedLamp1, Lamp1: footprint Resistor_THT:R_Axial_DIN0204_L3.6mm_D1.6mm_P5.08mm_Horizontal -> Resistor_THT:R_Axial_DIN0204_L3.6mm_D1.6mm_P2.54mm_Vertical
Connections:
- net GNDREF: now also InvertedLamp1.1 (-), Lamp1.1 (-)
- net at NPN2.1 (G), PNP2.1 (G): now also IC1.7 (OUTB), R4.1; no longer InvertedLamp1.1 (-)
- net at NPN1.1 (G), PNP1.1 (G): now also Auto/Man1.2, IC1.6 (VINB-), R3.1; no longer Lamp1.1 (-)
Other:
- moved on the sheet: Lamp1, R3
