File: HBroBil.kicad_pcb (KiCad board)
At the start: 2 copper layers, 13 parts, among them J1 Conn_01x07_Male

Commit message: Comparator component
Parts:
- removed ComperatorSocket1: Conn_02x04_Counter_Clockwise, Connector_PinSocket_1.27mm:PinSocket_2x04_P1.27mm_Vertical
- added IC1: MCP6542-I_P, MCP6542-I_P:DIP781W56P254L950H533Q8N, F.Cu at (132.1, 111.8)
- moved NPN2 17.8 mm to (156.5, 98.6), turned to 0 degrees
- moved R2 9.75 mm to (132.1, 101.1), turned to 180 degrees
- moved PNP2 7.69 mm to (169.2, 98.5), turned to 0 degrees
- moved R1 5.18 mm to (127.0, 95.5), turned to 0 degrees
Routing:
- net Net-(Auto/Man1-Pad2): track 37.8 -> 80.7 mm, vias 0 -> 2
- net /5V: track 75.4 -> 110.3 mm
- net /MTR -: track 98.2 -> 72.7 mm, vias 0 -> 2
- net /6V: track 123.0 -> 132.7 mm
- net Net-(NPN1-Pad3): track 282.0 -> 290.3 mm
- net Net-(IC1-Pad7): track 17.8 -> 20.5 mm
- net Net-(IC1-Pad5): track 20.0 -> 21.7 mm

Commit message: Finito
Parts:
- added FlybackNPN1: R_Small_US, Resistor_THT:R_Axial_DIN0204_L3.6mm_D1.6mm_P5.08mm_Horizontal, F.Cu at (144.5, 58.9)
- added FlybackNPN2: R_Small_US, Resistor_THT:R_Axial_DIN0204_L3.6mm_D1.6mm_P5.08mm_Horizontal, F.Cu at (144.5, 63.4)
- added FlybackPNP1: R_Small_US, Resistor_THT:R_Axial_DIN0204_L3.6mm_D1.6mm_P5.08mm_Horizontal, F.Cu at (131.1, 58.9)
- added FlybackPNP2: R_Small_US, Resistor_THT:R_Axial_DIN0204_L3.6mm_D1.6mm_P5.08mm_Horizontal, F.Cu at (131.1, 63.4)
- added InvertedLamp1: Lamp, Resistor_THT:R_Axial_DIN0204_L3.6mm_D1.6mm_P5.08mm_Horizontal, F.Cu at (152.4, 98.7)
- added Lamp1: Lamp, Resistor_THT:R_Axial_DIN0204_L3.6mm_D1.6mm_P5.08mm_Horizontal, F.Cu at (152.1, 113.8)
- added R3: R, Resistor_THT:R_Axial_DIN0204_L3.6mm_D1.6mm_P5.08mm_Horizontal, F.Cu at (139.1, 113.8)
- added R4: R, Resistor_THT:R_Axial_DIN0204_L3.6mm_D1.6mm_P5.08mm_Horizontal, F.Cu at (143.9, 108.8)
- moved NPN3 15.4 mm to (133.1, 126.3)
- moved PNP2 13.8 mm to (156.5, 93.0)
- moved NPN1 13.3 mm to (156.3, 111.3)
- moved PNP1 2.21 mm to (156.3, 105.6)
- moved R1 1.48 mm to (128.3, 96.3)
- moved ManDir1 1.42 mm to (111.6, 117.3)
- moved R2 1.33 mm to (133.3, 101.5), turned to 0 degrees
- moved PotentioMTR1 1.17 mm to (111.8, 94.2)
- turned IC1 to 90 degrees
- renumbered ManuelHastighed1 to PotentioMTR1
Connections:
- NPN1 pad 1: Net-(Auto/Man1-Pad2) -> Net-(NPN1-Pad1)
- NPN2 pad 1: Net-(IC1-Pad7) -> Net-(NPN2-Pad1)
- PNP1 pad 1: Net-(Auto/Man1-Pad2) -> Net-(NPN1-Pad1)
- PNP2 pad 1: Net-(IC1-Pad7) -> Net-(NPN2-Pad1)
Routing:
- net Net-(NPN1-Pad3): track 290.3 -> 105.4 mm
- net Net-(Auto/Man1-Pad2): track 80.7 -> 35.4 mm, vias 2 -> 0
- net /5V: track 110.3 -> 81.2 mm
- net Net-(HastighedSwitch1-Pad2): track 77.1 -> 97.8 mm
- net /MTR +: track 101.9 -> 86.3 mm
- net /MTR -: track 72.7 -> 60.1 mm
- net Net-(NPN1-Pad1): track 0.00 -> 10.9 mm
- net Net-(NPN2-Pad1): track 0.00 -> 9.72 mm
- net Net-(IC1-Pad5): track 21.7 -> 12.6 mm
- net Net-(InvertedLamp1-Pad2): track 0.00 -> 6.50 mm
- net Net-(IC1-Pad7): track 20.5 -> 15.6 mm
- net /SPD: track 46.1 -> 41.4 mm
- net /6V: track 132.7 -> 137.1 mm, vias 2 -> 0
- net /DIR: track 20.7 -> 17.5 mm
- net Net-(Lamp1-Pad2): track 0.00 -> 2.92 mm
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
Commit message: Fixed wire corners
Parts:
- moved HastighedSwitch1 6.71 mm to (111.7, 76.2)
- moved PotentioMTR1 5.33 mm to (111.8, 88.9)
Routing:
- net Net-(HastighedSwitch1-Pad2): track 97.8 -> 90.6 mm
- net /DIR: track 17.5 -> 10.8 mm
- net /6V: track 137.1 -> 131.8 mm
- net Net-(NPN1-Pad3): track 105.4 -> 102.4 mm
- net /MTR +: track 86.3 -> 88.6 mm
- net Net-(IC1-Pad7): track 15.6 -> 17.6 mm
- net /5V: track 81.2 -> 79.5 mm
- net Net-(HastighedSwitch1-Pad3): track 13.3 -> 14.7 mm

Commit message: Fixed wire Width, removed overlap connection
Routing:
- net /MTR -: track 60.1 -> 46.5 mm
- net /5V: track 79.5 -> 80.0 mm

Commit message: Moar Fixz
Connections:
- PotentioMTR1 pad 3: unconnected-(PotentioMTR1-Pad3) -> GNDREF
- R2 pad 2: GND -> GNDREF
Routing:
- net /6V: track 132.0 -> 130.8 mm
- added copper zone on F.Cu, net GNDREF
- removed copper zone on F.Cu, net GND

Commit message: fixs
Parts:
- moved R4 11.0 mm to (139.7, 98.7)
- turned InvertedLamp1 to 180 degrees
Routing:
- net Net-(IC1-Pad7): track 17.6 -> 24.1 mm
- net /6V: track 130.8 -> 125.9 mm
- net Net-(InvertedLamp1-Pad2): track 6.50 -> 2.57 mm
- net /MTR +: track 88.4 -> 89.3 mm

Commit message: lAST FIXES
Parts:
- FlybackNPN1, FlybackNPN2, FlybackPNP1, FlybackPNP2, R1, R2, R3, R4: footprint Resistor_THT:R_Axial_DIN0204_L3.6mm_D1.6mm_P5.08mm_Horizontal -> Resistor_THT:R_Axial_DIN0204_L3.6mm_D1.6mm_P7.62mm_Horizontal
- InvertedLamp1, Lamp1: footprint Resistor_THT:R_Axial_DIN0204_L3.6mm_D1.6mm_P5.08mm_Horizontal -> Resistor_THT:R_Axial_DIN0204_L3.6mm_D1.6mm_P2.54mm_Vertical
- moved HastighedSwitch1 14.7 mm to (111.6, 90.9)
- moved PotentioMTR1 12.2 mm to (111.8, 76.7)
- moved InvertedLamp1 7.37 mm to (147.3, 104.0), turned to 90 degrees
- moved FlybackNPN2 4.67 mm to (149.2, 63.4)
- moved FlybackNPN1 4.65 mm to (149.2, 59.0)
- moved R2 3.61 mm to (135.9, 104.0)
- moved Lamp1 0.13 mm to (152.3, 113.8)
- moved R4 0.13 mm to (139.7, 98.8)
Connections:
- Auto/Man1 pad 2: Net-(Auto/Man1-Pad2) -> Net-(NPN1-Pad1)
- IC1 pad 6: Net-(Auto/Man1-Pad2) -> Net-(NPN1-Pad1)
- InvertedLamp1 pad 1: Net-(InvertedLamp1-Pad1) -> GNDREF
- Lamp1 pad 1: Net-(Lamp1-Pad1) -> GNDREF
- NPN1 pad 1: Net-(Lamp1-Pad1) -> Net-(NPN1-Pad1)
- NPN2 pad 1: Net-(InvertedLamp1-Pad1) -> Net-(IC1-Pad7)
- PNP1 pad 1: Net-(Lamp1-Pad1) -> Net-(NPN1-Pad1)
- PNP2 pad 1: Net-(InvertedLamp1-Pad1) -> Net-(IC1-Pad7)
- R3 pad 1: Net-(Auto/Man1-Pad2) -> Net-(NPN1-Pad1)
Routing:
- net Net-(NPN1-Pad1): track 0.00 -> 59.8 mm
- net Net-(Auto/Man1-Pad2): track 35.8 -> 0.00 mm
- net Net-(HastighedSwitch1-Pad2): track 90.6 -> 67.6 mm
- net Net-(IC1-Pad7): track 24.1 -> 43.0 mm, vias 0 -> 2
- net /MTR +: track 89.3 -> 74.0 mm, vias 0 -> 2
- net /DIR: track 10.8 -> 25.5 mm
- net /6V: track 125.9 -> 111.8 mm
- net Net-(Lamp1-Pad1): track 10.9 -> 0.00 mm
- net Net-(InvertedLamp1-Pad1): track 9.72 -> 0.00 mm
- net Net-(FlybackNPN1-Pad1): track 102.4 -> 110.1 mm
- net /MTR -: track 46.4 -> 43.9 mm
- net Net-(HastighedSwitch1-Pad3): track 14.7 -> 16.2 mm
- net Net-(IC1-Pad5): track 12.6 -> 11.6 mm

Commit message: Thicc
Parts:
- moved InvertedLamp1 23.3 mm to (151.9, 126.8)
- moved R4 19.8 mm to (151.9, 114.4), turned to -90 degrees
- moved R2 14.9 mm to (146.6, 114.4), turned to -90 degrees
- moved Lamp1 13.4 mm to (149.2, 126.8), turned to 90 degrees
- moved R3 10.2 mm to (149.2, 114.4), turned to -90 degrees
Connections:
- Auto/Man1 pad 2: Net-(NPN1-Pad1) -> Net-(Auto/Man1-Pad2)
- NPN1 pad 1: Net-(NPN1-Pad1) -> Net-(Auto/Man1-Pad2)
- PNP1 pad 1: Net-(NPN1-Pad1) -> Net-(Auto/Man1-Pad2)
- R3 pad 1: Net-(NPN1-Pad1) -> Net-(Auto/Man1-Pad2)
Routing:
- net Net-(Auto/Man1-Pad2): track 0.00 -> 64.2 mm
- net Net-(NPN1-Pad1): track 59.8 -> 0.00 mm
- net Net-(IC1-Pad7): track 43.0 -> 71.6 mm
- net /MTR -: track 43.9 -> 62.2 mm
- net /MTR +: track 74.0 -> 89.1 mm
- net Net-(IC1-Pad5): track 11.6 -> 25.0 mm
- net /6V: track 111.8 -> 109.1 mm
- net Net-(Lamp1-Pad2): track 3.06 -> 2.24 mm
- net Net-(FlybackNPN1-Pad1): track 110.1 -> 109.5 mm
- net /5V: track 80.3 -> 79.8 mm
