File: HBroBil.kicad_pcb (KiCad board)
At the start: 2 copper layers, 21 parts, among them IC1 MCP6542-I_P, J1 Conn_01x07_Male

Commit message: Smol fix
Connections:
- IC1 pad 4: unconnected-(IC1-Pad4) -> GNDREF
- IC1 pad 6: Net-(NPN1-Pad1) -> Net-(Auto/Man1-Pad2)
Routing:
- net /6V: track 109.1 -> 111.3 mm
